Commit message: fixed wheel and caster  location

File: urdf/jambot_description.urdf.xacro (robot description, xacro)
@@ -13,5 +13,5 @@
   <xacro:property name="wheel_thickness" value="0.0265"/>
   <xacro:property name="wheel_mass" value="0.05"/>
-  <xacro:property name="wheel_offset_x" value="0.034"/>
+  <xacro:property name="wheel_offset_x" value="${chassis_length - 0.034}"/>
   <xacro:property name="wheel_offset_y" value="0.0865"/>
   <xacro:property name="wheel_offset_z" value="0.01"/>
@@ -19,5 +19,5 @@
   <xacro:property name="caster_wheel_radius" value="0.009"/>
   <xacro:property name="caster_wheel_mass" value="0.002"/>
-  <xacro:property name="caster_wheel_offset_x" value="0.12"/>
+  <xacro:property name="caster_wheel_offset_x" value="${chassis_length - 0.12}"/>
   <xacro:property name="caster_wheel_offset_z" value="${wheel_offset_z - wheel_radius + caster_wheel_radius}"/>
   <!-- Base Link -->

Commit message: removed the step from the camera

File: urdf/jambot_description.urdf.xacro (robot description, xacro)
@@ -144,10 +144,10 @@
     <parent link="${prefix}chassis"/>
     <child link="${prefix}camera_link"/>
-    <origin xyz="0.14 0 0.05" rpy="0 0 0"/>
+    <origin xyz="${chassis_length} 0 ${chassis_height/2}" rpy="0 0 0"/>
   </joint>
   <link name="${prefix}camera_link">
     <visual>
       <geometry>
-        <box size="0.010 0.03 0.03"/>
+        <box size="0.03 0.03 0.03"/>
       </geometry>
       <material name="black"/>

Commit message: fixed urdf and added slam config file

File: urdf/jambot_description.urdf.xacro (robot description, xacro)
@@ -164,5 +164,5 @@
     <parent link="${prefix}chassis"/>
     <child link="${prefix}laser_frame"/>
-    <origin xyz="0.085 0 0.105" rpy="0 0 0"/>
+    <origin xyz="0.085 0 0.105" rpy="0 0 ${PI}"/>
   </joint>
   <link name="${prefix}laser_frame">

Commit message: increased caster weight

File: urdf/jambot_description.urdf.xacro (robot description, xacro)
@@ -18,5 +18,5 @@
   <!-- Caster wheel properties -->
   <xacro:property name="caster_wheel_radius" value="0.009"/>
-  <xacro:property name="caster_wheel_mass" value="0.002"/>
+  <xacro:property name="caster_wheel_mass" value="0.02"/>
   <xacro:property name="caster_wheel_offset_x" value="${chassis_length - 0.12}"/>
   <xacro:property name="caster_wheel_offset_z" value="${wheel_offset_z - wheel_radius + caster_wheel_radius}"/>
@@ -173,11 +173,4 @@
       <material name="black"/>
     </visual>
-    <visual>
-      <origin xyz="0 0 -0.05"/>
-      <geometry>
-        <cylinder radius="0.01" length="0.1"/>
-      </geometry>
-      <material name="black"/>
-    </visual>
     <collision>
       <geometry>
@@ -187,5 +180,5 @@
     <inertial>
       <origin xyz="0 0 0" rpy="0 0 0"/>
-      <mass value="0.1"/>
+      <mass value="0.300"/>
       <inertia ixx="${(1/12) * 0.1 * (3*0.05*0.05 + 0.04*0.04)}" ixy="0.0" ixz="0.0"
               iyy="${(1/12) * 0.1 * (3*0.05*0.05 + 0.04*0.04)}" iyz="0.0"
