Commit message: Add EKF odom fusion, wire SLAM to filtered odom, and increase drive   speed limits

File: urdf/jambot_description.urdf.xacro (robot description, xacro)
@@ -160,4 +160,11 @@
   </joint>
   <link name="${prefix}camera_link_optical"/>
+  <!-- IMU -->
+  <joint name="${prefix}imu_joint" type="fixed">
+    <parent link="${prefix}base_link"/>
+    <child link="${prefix}imu_link"/>
+    <origin xyz="0.0 0.0 0.05" rpy="0 0 0"/>
+  </joint>
+  <link name="${prefix}imu_link"/>
   <!-- Lidar -->
   <joint name="${prefix}laser_joint" type="fixed">
