Commit message: added battery node and fixed direction

File: urdf/jambot.ros2_control.xacro (robot description, xacro)
@@ -27,4 +27,7 @@
         <state_interface name="velocity"/>
       </joint>
+      <sensor name="battery">
+        <state_interface name="voltage"/>
+      </sensor>
     </ros2_control>
   </xacro:macro>

File: urdf/jambot_description.urdf.xacro (robot description, xacro)
@@ -36,5 +36,5 @@
     <parent link="${prefix}base_link"/>
     <child link="${prefix}chassis"/>
-    <origin xyz="${-wheel_offset_x} 0 ${-wheel_offset_z}"/>
+    <origin xyz="${wheel_offset_x} 0 ${-wheel_offset_z}" rpy="0 0 ${PI}"/>
   </joint>
   <link name="${prefix}chassis">
